File: pcb/TodoPad.kicad_pcb (KiCad board)
At the start: 2 copper layers, 99 x 97.2 mm, 31 parts, among them SW1 SW_Push, SW10 SW_Push, SW11 SW_Push, SW12 SW_Push, SW13 SW_Push, SW14 SW_Push, SW2 SW_Push, SW3 SW_Push, SW4 SW_Push, SW5 SW_Push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

Commit message: Finalised everything
Parts:
- moved U2 0.61 mm to (120.9, 128.4)
Routing:
- net Net-(U1-GPIO7/SCL): track 99.2 -> 99.8 mm
- net +5V: track 102.6 -> 103.3 mm
- net Net-(U1-GPIO6/SDA): track 104.4 -> 105.0 mm
Changed lines of the file:
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@@
 	(footprint "4-pin SSD1306 OLED 128x32:SSD1306-0.91-OLED-4pin-128x32"
 		(layer "F.Cu")
-		(at 120.2975 128.48625)
+		(at 120.9 128.4)
 		(property "Reference" "U2"
 			(at 1.9 5.91 90)
@@
 	)
 	(segment
+		(start 142.4265 118.84525)
+		(end 142.4265 64.78519)
+		(width 0.2)
+		(layer "F.Cu")
+		(net 24)
+	)
+	(segment
+		(start 142.4265 64.78519)
+		(end 146.36219 60.8495)
+		(width 0.2)
+		(layer "F.Cu")
+		(net 24)
+	)
+	(segment
+		(start 146.36219 55.3555)
+		(end 145.7395 54.73281)
+		(width 0.2)
+		(layer "F.Cu")
+		(net 24)
+	)
+	(segment
+		(start 156.7975 133.21625)
+		(end 142.4265 118.84525)
+		(width 0.2)
+		(layer "F.Cu")
+		(net 24)
+	)
+	(segment
+		(start 153.150763 58.150763)
+		(end 150.3555 55.3555)
+		(width 0.2)
+		(layer "F.Cu")
+		(net 24)
+	)
+	(segment
+		(start 150.3555 55.3555)
+		(end 146.36219 55.3555)
+		(width 0.2)
+		(layer "F.Cu")
+		(net 24)
+	)
+	(segment
 		(start 145.7395 50.2755)
 		(end 146.8025 49.2125)
@@
 	)
 	(segment
-		(start 142.4265 118.84525)
-		(end 142.4265 64.78519)
-		(width 0.2)
-		(layer "F.Cu")
-		(net 24)
-	)
-	(segment
 		(start 150.452026 60.8495)
 		(end 153.150763 58.150763)
@@
 	)
 	(segment
-		(start 153.150763 58.150763)
-		(end 150.3555 55.3555)
+		(start 157.31375 133.21625)
+		(end 156.7975 133.21625)
 		(width 0.2)
 		(layer "F.Cu")
@@
 	)
 	(segment
-		(start 142.4265 64.78519)
-		(end 146.36219 60.8495)
-		(width 0.2)
-		(layer "F.Cu")
-		(net 24)
-	)
-	(segment
-		(start 146.36219 55.3555)
-		(end 145.7395 54.73281)
-		(width 0.2)
-		(layer "F.Cu")
-		(net 24)
-	)
-	(segment
-		(start 150.3555 55.3555)
-		(end 146.36219 55.3555)
+		(start 145.7395 54.73281)
+		(end 145.7395 50.2755)
 		(width 0.2)
 		(layer "F.Cu")
@@
 	)
 	(segment
-		(start 156.7975 133.21625)
-		(end 142.4265 118.84525)
+		(start 157.4 133.13)
+		(end 157.31375 133.21625)
 		(width 0.2)
 		(layer "F.Cu")
@@
 	)
 	(segment
-		(start 145.7395 54.73281)
-		(end 145.7395 50.2755)
-		(width 0.2)
-		(layer "F.Cu")
-		(net 24)
+		(start 128.409128 113.878436)
+		(end 126.427814 115.85975)
+		(width 0.2)
+		(layer "F.Cu")
+		(net 25)
+	)
+	(segment
+		(start 134.919686 113.878436)
+		(end 128.409128 113.878436)
+		(width 0.2)
+		(layer "F.Cu")
+		(net 25)
+	)
+	(segment
+		(start 157.31375 135.75625)
+		(end 156.7975 135.75625)
+		(width 0.2)
+		(layer "F.Cu")
+		(net 25)
+	)
+	(segment
+		(start 126.427814 115.85975)
+		(end 125.267186 115.85975)
+		(width 0.2)
+		(layer "F.Cu")
+		(net 25)
 	)
 	(segment
@@
 	)
 	(segment
+		(start 156.7975 135.75625)
+		(end 134.919686 113.878436)
+		(width 0.2)
+		(layer "F.Cu")
+		(net 25)
+	)
+	(segment
 		(start 123.3765 113.969064)
 		(end 123.3765 69.2635)
@@
 	)
 	(segment
-		(start 156.7975 135.75625)
-		(end 134.919686 113.878436)
-		(width 0.2)
-		(layer "F.Cu")
-		(net 25)
-	)
-	(segment
-		(start 134.919686 113.878436)
-		(end 128.409128 113.878436)
-		(width 0.2)
-		(layer "F.Cu")
-		(net 25)
-	)
-	(segment
-		(start 128.409128 113.878436)
-		(end 126.427814 115.85975)
+		(start 157.4 135.67)
+		(end 157.31375 135.75625)
 		(width 0.2)
 		(layer "F.Cu")
@@
 	)
 	(segment
-		(start 126.427814 115.85975)
-		(end 125.267186 115.85975)
-		(width 0.2)
-		(layer "F.Cu")
-		(net 25)
+		(start 157.6 130.39)
+		(end 157.4 130.59)
+		(width 0.2)
+		(layer "F.Cu")
+		(net 26)
+	)
+	(segment
+		(start 157.6 129.87375)
+		(end 157.6 130.39)
+		(width 0.2)
+		(layer "F.Cu")
+		(net 26)
+	)
+	(segment
+		(start 146.8025 51.7525)
+		(end 160.372564 51.7525)
+		(width 0.2)
+		(layer "F.Cu")
+		(net 26)
+	)
+	(segment
+		(start 160.372564 51.7525)
+		(end 165.3485 56.728436)
+		(width 0.2)
+		(layer "F.Cu")
+		(net 26)
 	)
 	(segment
@@
 	)
 	(segment
-		(start 160.372564 51.7525)
-		(end 165.3485 56.728436)
+		(start 165.3485 122.12525)
+		(end 157.6 129.87375)
 		(width 0.2)
 		(layer "F.Cu")
@@
 	)
 	(segment
-		(start 146.8025 51.7525)
-		(end 160.372564 51.7525)
-		(width 0.2)
-		(layer "F.Cu")
-		(net 26)
-	)
-	(segment
-		(start 165.3485 122.12525)
-		(end 156.7975 130.67625)
-		(width 0.2)
-		(layer "F.Cu")
-		(net 26)
+		(start 157.4 138.21)
+		(end 157.31375 138.29625)
+		(width 0.2)
+		(layer "F.Cu")
+		(net 28)
 	)
 	(segment
@@
 	)
 	(segment
+		(start 157.31375 138.29625)
+		(end 144.17653 138.29625)
+		(width 0.2)
+		(layer "F.Cu")
+		(net 28)
+	)
+	(segment
+		(start 122.9755 117.09522)
+		(end 122.9755 67.1245)
+		(width 0.2)
+		(layer "F.Cu")
+		(net 28)
+	)
+	(segment
 		(start 144.17653 138.29625)
 		(end 122.9755 117.09522)
 		(width 0.2)
 		(layer "F.Cu")
-		(net 28)
-	)
-	(segment
-		(start 122.9755 117.09522)
-		(end 122.9755 67.1245)
-		(width 0.2)
-		(layer "F.Cu")
-		(net 28)
-	)
-	(segment
-		(start 156.7975 138.29625)
-		(end 144.17653 138.29625)
-		(width 0.2)
-		(layer "F.Cu")

Commit message: Modified PCB for production
Parts:
- removed the G*** at (184.5, 138.0)
- added G***: LOGO, Icons:wolfIconLarge, F.Cu at (181.9, 136.8)
